File: pathfinder.kicad_sch (KiCad schematic)
At the start: 31 parts, among them J1 Conn_01x04, SW1 SW_Push, SW2 SW_Push, SW3 SW_Push, SW4 SW_Push, SW5 SW_Push, SW6 SW_Push, SW7 SW_Push, SW8 SW_Push, SW9 SW_Push, U1 XIAO-RP2040-DIP

Commit message: work
Parts:
- removed C1: 100uF, Capacitor_SMD:CP_Elec_5x5.3, symbol Device:C_Polarized
- removed J1: Conn_01x04, Connector_PinHeader_2.54mm:PinHeader_1x04_P2.54mm_Vertical, symbol Connector_Generic:Conn_01x04
- removed R1: 330R, Resistor_SMD:R_0805_2012Metric, symbol Device:R
- added U2: OLED_0.91_128x32, Hackclub Footprints:OLED_0.91_128x32, symbol Hackclub Symbols:OLED_0.91_128x32
Connections:
- net DIN1: now also U1.7 (GPIO0/TX)
- net GND: now also U2.1 (GND)
- net SCL: now also U2.3 (SCL)
- net SDA: now also U2.4 (SDA)
- net VCC: now also U2.2 (VCC)
