File: pathfinder.kicad_pcb (KiCad board)
At the start: 2 copper layers, 30 parts, among them SW1 SW_Push, SW2 SW_Push, SW3 SW_Push, SW4 SW_Push, SW5 SW_Push, SW6 SW_Push, SW7 SW_Push, SW8 SW_Push, SW9 SW_Push, U1 XIAO-RP2040-DIP

Commit message: work
Parts:
- removed C1: 100uF, Capacitor_SMD:CP_Elec_5x5.3
- removed R1: 330R, Resistor_SMD:R_0805_2012Metric
- added U2: OLED_0.91_128x32, Hackclub Footprints:OLED_0.91_128x32, F.Cu at (101.6, 79.6)
- D1, D2, D3, D4, D5, D6, D7, D8, D9: footprint Diode_SMD:D_SOD-123 -> Diode_THT:D_DO-35_SOD27_P7.62mm_Horizontal; moved to B.Cu
- D10, D11, D12, D13, D14, D15, D16, D17, D18: value WS2812B -> SK6812MINI-E; footprint LED_SMD:LED_WS2812B_PLCC4_5.0x5.0mm_P3.2mm -> Hackclub Footprints:MX_SK6812MINI-E_REV
- U1: moved to B.Cu
- moved D7 177.4 mm to (91.9, 143.2)
- moved D4 164.5 mm to (91.8, 124.1)
- moved D8 163.4 mm to (109.6, 143.1)
- moved D5 150.2 mm to (109.5, 124.1)
- moved D9 148.2 mm to (128.6, 143.1)
- moved D2 139.0 mm to (109.5, 105.1)
- moved D6 134.6 mm to (128.6, 124.0)
- moved D16 130.9 mm to (100.0, 138.1)
- moved D13 124.5 mm to (100.0, 119.0)
- moved D3 123.3 mm to (128.6, 105.0)
- moved D10 121.2 mm to (100.0, 100.0)
- moved D17 112.1 mm to (119.0, 138.1)
- moved D14 107.2 mm to (119.0, 119.0)
- moved D11 106.0 mm to (119.0, 100.0)
- moved D18 93.9 mm to (138.1, 138.1)
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Connections:
- U1 pad 10: unconnected-(U1-GPIO4/MISO-Pad10) -> COL3
- U1 pad 12: unconnected-(U1-3V3-Pad12) -> VCC
- U1 pad 5: COL2 -> SDA
- U1 pad 6: COL3 -> SCL
- U1 pad 7: Net-(U1-GPIO0/TX) -> DIN1
- U1 pad 9: unconnected-(U1-GPIO2/SCK-Pad9)_1 -> COL2
Routing:
- net ROW2: track 0.00 -> 166.9 mm, vias 0 -> 4
- net ROW3: track 0.00 -> 132.4 mm, vias 0 -> 6
- net ROW1: track 0.00 -> 87.4 mm
- net COL3: track 0.00 -> 84.6 mm, vias 0 -> 1
- net Net-(D15-DOUT): track 0.00 -> 62.5 mm
- net Net-(D12-DOUT): track 0.00 -> 60.3 mm
- net COL2: track 0.00 -> 59.4 mm, vias 0 -> 1
- net DIN1: track 0.00 -> 44.3 mm
- net COL1: track 0.00 -> 38.1 mm
- net Net-(D11-DOUT): track 0.00 -> 14.8 mm
- net Net-(D13-DOUT): track 0.00 -> 14.8 mm
- net Net-(D14-DOUT): track 0.00 -> 14.8 mm
- net Net-(D17-DOUT): track 0.00 -> 14.8 mm
- net Net-(D10-DOUT): track 0.00 -> 14.8 mm
- net Net-(D16-DOUT): track 0.00 -> 14.7 mm
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Other:
- board outline added: 90.5 x 114.3 mm

Commit message: work
Routing:
- net VBUS: track 0.00 -> 206.7 mm, vias 0 -> 10
- net GND: track 7.93 -> 86.0 mm, vias 1 -> 5
- net COL1: track 38.1 -> 70.6 mm, vias 0 -> 2
- net ROW1: track 87.4 -> 82.8 mm
- net ROW2: track 166.9 -> 167.6 mm
- added copper zone on B.Cu, net GND
Other:
- board size 90.5 x 114.3 mm -> 60.5 x 86 mm

Commit message: dxfcgvhbjn
Routing:
- net GND: track 86.0 -> 29.2 mm, vias 5 -> 1
- net ROW1: track 82.8 -> 92.6 mm
- net VBUS: track 206.7 -> 209.0 mm
- net (no net): vias 0 -> 4
