File: pommepad/pommepad.kicad_pcb (KiCad board)
At the start: 2 copper layers, 90.9 x 76.6 mm, 20 parts, among them SW1 SW_Push, SW2 SW_Push, SW3 SW_Push, SW4 SW_Push, SW5 SW_Push, SW6 SW_Push, U1 XIAO-RP2040-DIP, U2 OLED_0.91_128x32

Commit message: war is over.
I FINISHED THE PCB IM IN TEARS BRO
Parts:
- added G***: LOGO, LOGO, F.Cu at (185.3, 132.7)
- added G***: LOGO, LOGO, F.Cu at (234.1, 92.9)
- added G***: LOGO, LOGO, F.Cu at (209.8, 131.2)
- added REF**: MountingHole_3mm, MountingHole:MountingHole_3mm, F.Cu at (235.6, 83.8)
- added REF**: MountingHole_3mm, MountingHole:MountingHole_3mm, F.Cu at (159.4, 105.3)
- added REF**: MountingHole_3mm, MountingHole:MountingHole_3mm, F.Cu at (235.6, 102.9)
- added REF**: MountingHole_3mm, MountingHole:MountingHole_3mm, F.Cu at (159.4, 83.8)
- moved D1 44.1 mm to (169.7, 102.4)
- moved D12 44.1 mm to (179.1, 120.8)
- moved D4 44.1 mm to (169.7, 121.5)
- moved D6 44.1 mm to (207.9, 121.3)
- moved D8 44.1 mm to (198.3, 101.6)
- moved SW1 44.1 mm to (179.3, 97.2)
- moved SW2 44.1 mm to (198.3, 97.2)
- moved SW4 44.1 mm to (179.3, 116.3)
- moved SW5 44.1 mm to (198.3, 116.3)
- moved SW6 44.1 mm to (217.4, 116.2)
- moved U2 44.1 mm to (191.4, 78.6)
- moved D2 44.1 mm to (188.8, 102.4)
- moved D3 44.1 mm to (207.8, 102.5)
- moved D9 44.1 mm to (217.5, 101.7)
- moved D10 44.1 mm to (217.4, 120.6)
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Routing:
- net GND: track 64.0 -> 38.4 mm, vias 14 -> 8
- net COL3: track 76.1 -> 71.4 mm, vias 1 -> 0
- net 5V: track 153.8 -> 151.5 mm
- net (no net): vias 2 -> 1
Other:
- board text added: "but i like u more ;)"
- board text added: "i like apples! -->"
