File: pommepad/pommepad.kicad_sch (KiCad schematic)
At the start: 20 parts, among them SW1 SW_Push, SW2 SW_Push, SW3 SW_Push, SW4 SW_Push, SW5 SW_Push, SW6 SW_Push, U1 XIAO-RP2040-DIP, U2 OLED_0.91_128x32

Commit message: war is over.
I FINISHED THE PCB IM IN TEARS BRO
Connections:
- net 5V renamed +5V
